File: console_thing.kicad_pcb (KiCad board)
At the start: 2 copper layers, 74.5 x 30.7 mm, 74 parts, among them J1 Conn_01x03, SW1 SW_Push_45deg, SW2 SW_Push_45deg, SW3 SW_Push_45deg, SW4 SW_Push_45deg, SW5 SW_Push_45deg, SW6 SW_Push_45deg, SW7 SW_SPDT, U2 CH32V003FxPx

Commit message: reroute
Parts:
- SW7: moved to B.Cu
- U2: moved to F.Cu
- moved U2 53.4 mm to (189.2, 48.8)
- moved C1 50.9 mm to (194.8, 43.8), turned to 180 degrees
- moved H2 47.9 mm to (138.1, 60.0)
- moved SW5 46.9 mm to (125.1, 59.3)
- moved SW6 41.4 mm to (125.1, 66.9)
- moved J1 36.6 mm to (198.7, 40.2), turned to 180 degrees
- moved D5 35.6 mm to (132.9, 64.7)
- moved SW7 35.6 mm to (189.5, 40.5), turned to 0 degrees
- moved D17 35.4 mm to (168.2, 41.4)
- moved D25 35.4 mm to (168.2, 43.4)
- moved D33 35.3 mm to (168.2, 45.5)
- moved D41 35.3 mm to (168.2, 47.6)
- moved D49 35.3 mm to (168.2, 49.7)
- moved D57 35.2 mm to (168.2, 51.8)
- moved D65 35.2 mm to (168.2, 53.9)
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Connections:
- U2 pad 1: /Col2 -> unconnected-(U2-PD4-Pad1)
- U2 pad 10: /Row1 -> /LED0
- U2 pad 11: /LED0 -> /LED1
- U2 pad 12: /LED1 -> /LED2
- U2 pad 13: /LED2 -> /LED3
- U2 pad 14: /LED3 -> /LED4
- U2 pad 15: /LED4 -> /LED5
- U2 pad 16: /LED5 -> /LED6
- U2 pad 17: /LED6 -> /LED7
- U2 pad 19: /LED7 -> /USB D+
- U2 pad 2: /Col0 -> unconnected-(U2-PD5-Pad2)
- U2 pad 20: /Row0 -> /USB D-
- U2 pad 3: /Col1 -> unconnected-(U2-PD6-Pad3)
Routing:
- net /Row0: track 76.0 -> 0.00 mm, vias 2 -> 0
- net /Row1: track 67.8 -> 0.00 mm, vias 2 -> 0
- net /Col1: track 65.2 -> 0.00 mm, vias 1 -> 0
- net /Col2: track 54.6 -> 0.00 mm, vias 2 -> 0
- net /Col0: track 52.9 -> 0.00 mm, vias 1 -> 0
- net /LED1: track 79.3 -> 40.5 mm
- net /LED2: track 75.6 -> 39.6 mm
- net /LED3: track 72.5 -> 39.2 mm
- net GND: track 33.9 -> 3.27 mm
- net /LED4: track 70.3 -> 40.0 mm
- net /LED6: track 63.3 -> 36.3 mm
- net /LED5: track 67.6 -> 41.0 mm
- net /LED7: track 66.6 -> 45.6 mm
- net Net-(D6-A): track 18.1 -> 0.00 mm
- net /SWIO: track 32.0 -> 16.2 mm, vias 0 -> 1
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Other:
- board outline removed
- board text removed: "<3 Discord @funnsam Github @funnsam Website https://funn.is-a.dev/"

Commit message: rerouted
Parts:
- added BT1: Battery_Cell, Battery:BatteryHolder_Keystone_1058_1x2032, B.Cu at (194.3, 78.6)
- C1: value 100nF -> 0.1uF
- U2: moved to B.Cu
- moved SW5 97.3 mm to (220.7, 77.1), turned to 90 degrees
- moved D5 91.7 mm to (222.1, 86.0)
- moved SW6 90.2 mm to (214.2, 80.6), turned to 90 degrees
- moved D6 87.4 mm to (218.5, 85.4), turned to 90 degrees
- moved SW1 62.9 mm to (171.1, 71.8)
- moved SW3 62.7 mm to (177.6, 78.3), turned to 180 degrees
- moved SW2 57.5 mm to (164.6, 78.3)
- moved SW4 56.7 mm to (171.1, 84.8)
- moved D3 53.9 mm to (183.6, 77.0), turned to 90 degrees
- moved D4 50.6 mm to (178.0, 84.6), turned to -135 degrees
- moved J1 49.9 mm to (227.8, 80.8), turned to 0 degrees
- moved D1 49.8 mm to (177.8, 74.1), turned to 180 degrees
- moved SW7 44.7 mm to (226.3, 65.9)
- moved D2 44.7 mm to (170.6, 79.6), turned to -90 degrees
- moved C1 42.5 mm to (217.4, 79.8), turned to -90 degrees
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Connections:
- D3 pad 1: /Row1 -> /Row0
- D5 pad 1: /Row0 -> /Row1
- J1 pad 1: Net-(J1-Pin_1) -> +3V0
- SW3 pad 1: /Col0 -> /Col2
- SW4 pad 1: /Col1 -> /Col0
- SW5 pad 1: /Col2 -> /Col1
- SW7 pad 1: unconnected-(SW7-A-Pad1) -> +3V0
- SW7 pad 2: Net-(J1-Pin_1) -> Net-(BT1-+)
- SW7 pad 3: +3V0 -> unconnected-(SW7-C-Pad3)
- U2 pad 1: unconnected-(U2-PD4-Pad1) -> /Row0
- U2 pad 10: /LED0 -> /LED7
- U2 pad 11: /LED1 -> /LED6
- U2 pad 12: /LED2 -> /LED5
- U2 pad 13: /LED3 -> /LED4
- U2 pad 14: /LED4 -> /LED3
- U2 pad 15: /LED5 -> /LED2
- U2 pad 16: /LED6 -> /LED1
- U2 pad 17: /LED7 -> /LED0
- U2 pad 19: /USB D+ -> /Row1
- U2 pad 2: unconnected-(U2-PD5-Pad2) -> /Col0
- U2 pad 20: /USB D- -> /Col2
- U2 pad 3: unconnected-(U2-PD6-Pad3) -> /Col1
Routing:
- net /Col1: track 0.00 -> 88.0 mm, vias 0 -> 5
- net /Col0: track 0.00 -> 77.9 mm, vias 0 -> 3
- net /Row1: track 0.00 -> 61.3 mm, vias 0 -> 3
- net /Col2: track 0.00 -> 60.5 mm, vias 0 -> 1
- net /Row0: track 0.00 -> 55.5 mm, vias 0 -> 1
- net GND: track 3.27 -> 53.5 mm, vias 0 -> 2
- net Net-(BT1-+): track 0.00 -> 22.8 mm
- net +3V0: track 5.99 -> 26.5 mm, vias 1 -> 2
- net Net-(D5-A): track 0.00 -> 13.0 mm
- net Net-(D4-A): track 0.00 -> 10.9 mm
- net Net-(J1-Pin_1): track 10.4 -> 0.00 mm
- net Net-(D2-A): track 0.00 -> 9.97 mm
- net Net-(D6-A): track 0.00 -> 9.96 mm
- net Net-(D3-A): track 0.00 -> 9.95 mm
- net Net-(D1-A): track 0.00 -> 9.75 mm
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Other:
- board outline added: 75 x 30 mm

Commit message: updat
Parts:
- added H3: MountingHole, MountingHole:MountingHole_2.2mm_M2, F.Cu at (222.0, 77.0)
- moved H2 29.2 mm to (153.0, 77.0)
- moved H1 28.5 mm to (153.0, 53.0)
- moved SW7 16.7 mm to (216.8, 52.2)
- moved BT1 15.3 mm to (187.5, 65.0)
- moved D11 15.3 mm to (184.4, 58.7)
- moved D13 15.3 mm to (188.6, 58.7)
- moved D15 15.3 mm to (192.8, 58.7)
- moved D17 15.3 mm to (180.2, 58.7)
- moved D5 15.3 mm to (215.3, 72.4)
- moved D65 15.3 mm to (180.2, 71.3)
- moved D67 15.3 mm to (184.4, 71.3)
- moved D69 15.3 mm to (188.6, 71.3)
- moved D71 15.3 mm to (192.8, 71.3)
- moved J1 15.3 mm to (221.0, 67.1)
- moved SW5 15.3 mm to (213.9, 63.4)
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Connections:
- J1 pad 1: +3V0 -> Net-(J1-Pin_1)
- SW7 pad 1: +3V0 -> Net-(BT1-+)
- SW7 pad 2: Net-(BT1-+) -> +3V0
- SW7 pad 3: unconnected-(SW7-C-Pad3) -> Net-(J1-Pin_1)
Routing:
- net Net-(J1-Pin_1): track 0.00 -> 13.1 mm, vias 0 -> 1
- net Net-(BT1-+): track 22.8 -> 16.6 mm
- net +3V0: track 26.5 -> 23.3 mm
- added copper zone on B.Cu, net GND
- added copper zone on F.Cu, net GND
Other:
- outline, holes or cut-outs redrawn
